Commit message: xzfxccxz

File: description/robot_core.xacro (robot description, xacro)
@@ -20,5 +20,5 @@
         <origin xyz="0.1 0 0"/>
     </joint>
-    <link name="chassin">
+    <link name="chassis">
         <visual>
             <origin xyz= "0.15 0 0.075"/>

Commit message: 132

File: description/robot_core.xacro (robot description, xacro)
@@ -18,9 +18,9 @@
         <parent link="base_link"/>
         <child link="chassis"/>
-        <origin xyz="0.1 0 0"/>
+        <origin xyz="0 0 0"/>
     </joint>
     <link name="chassis">
         <visual>
-            <origin xyz= "0.15 0 0.075"/>
+            <origin xyz= "0 0 0.075"/>
             <geometry>
                 <box size="0.3 0.3 0.15"/>
@@ -29,3 +29,4 @@
         </visual>
     </link>
+# gojkhp'ijdsfhpoij
 </robot>

Commit message: -1

File: description/robot_core.xacro (robot description, xacro)
@@ -18,5 +18,5 @@
         <parent link="base_link"/>
         <child link="chassis"/>
-        <origin xyz="0 0 0"/>
+        <origin xyz="0 0 -1"/>
     </joint>
     <link name="chassis">
@@ -29,4 +29,3 @@
         </visual>
     </link>
-# gojkhp'ijdsfhpoij
 </robot>

Commit message: gotovo

File: description/robot_core.xacro (robot description, xacro)
@@ -18,9 +18,9 @@
         <parent link="base_link"/>
         <child link="chassis"/>
-        <origin xyz="0 0 -1"/>
+        <origin xyz="-0.1 0 0"/>
     </joint>
     <link name="chassis">
         <visual>
-            <origin xyz= "0 0 0.075"/>
+            <origin xyz="0.15 0 0.075"/>
             <geometry>
                 <box size="0.3 0.3 0.15"/>

Commit message: pisi kolisa

File: description/robot_core.xacro (robot description, xacro)
@@ -29,3 +29,31 @@
         </visual>
     </link>
+    <joint name="left_wheel_joint" type="continuous">
+       <parent link="base_link"/>
+       <child link="left_wheel"/>
+       <origin xyz="0 0.175 0" rpy="${pi/2} 0 0"/>
+       <axis xyz="0 0 1"/>
+    </joint>
+    <link name="left_wheel">
+        <visual>
+            <geometry>
+                <cylinder radius="0.5" length="0.04"/>
+            </geometry>
+            <material name="blue"/>
+        </visual>
+    </link>
+    <joint name="right_wheel_joint" type="continuous">
+       <parent link="base_link"/>
+       <child link="right_wheel"/>
+       <origin xyz="0 -0.175 0" rpy="${pi/2} 0 0"/>
+       <axis xyz="0 0 -1"/>
+    </joint>
+    <link name="right_wheel">
+        <visual>
+            <geometry>
+                <cylinder radius="0.5" length="0.04"/>
+            </geometry>
+            <material name="blue"/>
+        </visual>
+    </link>
 </robot>

Commit message: pizda

File: description/robot_core.xacro (robot description, xacro)
@@ -38,5 +38,5 @@
         <visual>
             <geometry>
-                <cylinder radius="0.5" length="0.04"/>
+                <cylinder radius="0.05" length="0.04"/>
             </geometry>
             <material name="blue"/>
@@ -52,5 +52,5 @@
         <visual>
             <geometry>
-                <cylinder radius="0.5" length="0.04"/>
+                <cylinder radius="0.05" length="0.04"/>
             </geometry>
             <material name="blue"/>

Commit message: men

File: description/robot_core.xacro (robot description, xacro)
@@ -29,28 +29,30 @@
         </visual>
     </link>
+    <!-- LEFT WHEEL -->
     <joint name="left_wheel_joint" type="continuous">
-       <parent link="base_link"/>
-       <child link="left_wheel"/>
-       <origin xyz="0 0.175 0" rpy="${pi/2} 0 0"/>
-       <axis xyz="0 0 1"/>
+        <parent link="base_link"/>
+        <child link="left_wheel"/>
+        <origin xyz="0 0.175 0" rpy="-${pi/2} 0 0"/>
+        <axis xyz="0 0 1"/>
     </joint>
     <link name="left_wheel">
         <visual>
             <geometry>
-                <cylinder radius="0.05" length="0.04"/>
+                <cylinder length="0.04" radius="0.05" />
             </geometry>
             <material name="blue"/>
         </visual>
     </link>
+    <!-- RIGHT WHEEL -->
     <joint name="right_wheel_joint" type="continuous">
-       <parent link="base_link"/>
-       <child link="right_wheel"/>
-       <origin xyz="0 -0.175 0" rpy="${pi/2} 0 0"/>
-       <axis xyz="0 0 -1"/>
+        <parent link="base_link"/>
+        <child link="right_wheel"/>
+        <origin xyz="0 -0.175 0" rpy="${pi/2} 0 0"/>
+        <axis xyz="0 0 -1"/>
     </joint>
     <link name="right_wheel">
         <visual>
             <geometry>
-                <cylinder radius="0.05" length="0.04"/>
+                <cylinder length="0.04" radius="0.05" />
             </geometry>
             <material name="blue"/>

Commit message: pete

File: description/robot_core.xacro (robot description, xacro)
@@ -59,3 +59,17 @@
         </visual>
     </link>
+    <!-- CASTER WHEEL -->
+    <joint name="caster_wheel_joint" type="fixed">
+        <parent link="chassis"/>
+        <child link="caster_wheel"/>
+        <origin xyz="0.24 0 0" rpy="0 0 0"/>
+    </joint>
+    <link name="caster_wheel">
+        <visual>
+            <geometry>
+                <sphere radius="0.05" />
+            </geometry>
+            <material name="black"/>
+        </visual>
+    </link>
 </robot>

Commit message: CASTER WHEEL

File: description/robot_core.xacro (robot description, xacro)
@@ -73,3 +73,17 @@
         </visual>
     </link>
+    <!-- CASTER WHEEL -->
+    <joint name="caster_wheel_joint" type="fixed">
+        <parent link="chassis"/>
+        <child link="caster_wheel"/>
+        <origin xyz="0.24 0 0" rpy="0 0 0"/>
+    </joint>
+    <link name="caster_wheel">
+        <visual>
+            <geometry>
+                <sphere radius="0.05" />
+            </geometry>
+            <material name="black"/>
+        </visual>
+    </link>
 </robot>

Commit message: Короче

File: description/robot_core.xacro (robot description, xacro)
@@ -73,17 +73,3 @@
         </visual>
     </link>
-    <!-- CASTER WHEEL -->
-    <joint name="caster_wheel_joint" type="fixed">
-        <parent link="chassis"/>
-        <child link="caster_wheel"/>
-        <origin xyz="0.24 0 0" rpy="0 0 0"/>
-    </joint>
-    <link name="caster_wheel">
-        <visual>
-            <geometry>
-                <sphere radius="0.05" />
-            </geometry>
-            <material name="black"/>
-        </visual>
-    </link>
 </robot>

Commit message: Adding collision

File: description/robot_core.xacro (robot description, xacro)
@@ -73,3 +73,18 @@
         </visual>
     </link>
+    <link name="chassis">
+        <visual>
+            <origin xyz="0.15 0 0.075" rpy="0 0 0"/>
+            <geometry>
+                <box size="0.3 0.3 0.15"/>
+            </geometry>
+            <material name="white"/>
+        </visual>
+        <collision>
+            <origin xyz="0.15 0 0.075" rpy="0 0 0"/>
+            <geometry>
+                <box size="0.3 0.3 0.15"/>
+            </geometry>
+        </collision>
+    </link>
 </robot>

Commit message: fix: adding collision in chassis

File: description/robot_core.xacro (robot description, xacro)
@@ -22,5 +22,5 @@
     <link name="chassis">
         <visual>
-            <origin xyz="0.15 0 0.075"/>
+            <origin xyz="0.15 0 0.075" rpy="0 0 0"/>
             <geometry>
                 <box size="0.3 0.3 0.15"/>
@@ -28,4 +28,10 @@
             <material name="white"/>
         </visual>
+        <collision>
+            <origin xyz="0.15 0 0.075" rpy="0 0 0"/>
+            <geometry>
+                <box size="0.3 0.3 0.15"/>
+            </geometry>
+        </collision>
     </link>
     <!-- LEFT WHEEL -->
@@ -73,18 +79,2 @@
         </visual>
     </link>
-    <link name="chassis">
-        <visual>
-            <origin xyz="0.15 0 0.075" rpy="0 0 0"/>
-            <geometry>
-                <box size="0.3 0.3 0.15"/>
-            </geometry>
-            <material name="white"/>
-        </visual>
-        <collision>
-            <origin xyz="0.15 0 0.075" rpy="0 0 0"/>
-            <geometry>
-                <box size="0.3 0.3 0.15"/>
-            </geometry>
-        </collision>
-    </link>
-</robot>

Commit message: chassispuuppu

File: description/robot_core.xacro (robot description, xacro)
@@ -22,5 +22,5 @@
     <link name="chassis">
         <visual>
-            <origin xyz="0.15 0 0.075"/>
+            <origin xyz="0.15 0 0.075" rpy="0 0 0"/>
             <geometry>
                 <box size="0.3 0.3 0.15"/>
@@ -28,4 +28,10 @@
             <material name="white"/>
         </visual>
+        <collision>
+            <origin xyz="0.15 0 0.075" rpy="0 0 0"/>
+            <geometry>
+                <box size="0.3 0.3 0.15"/>
+            </geometry>
+        </collision>
     </link>
     <!-- LEFT WHEEL -->
@@ -73,18 +79,3 @@
         </visual>
     </link>
-    <link name="chassis">
-        <visual>
-            <origin xyz="0.15 0 0.075" rpy="0 0 0"/>
-            <geometry>
-                <box size="0.3 0.3 0.15"/>
-            </geometry>
-            <material name="white"/>
-        </visual>
-        <collision>
-            <origin xyz="0.15 0 0.075" rpy="0 0 0"/>
-            <geometry>
-                <box size="0.3 0.3 0.15"/>
-            </geometry>
-        </collision>
-    </link>
 </robot>

Commit message: feat: inercial in links

File: description/robot_core.xacro (robot description, xacro)
@@ -35,4 +35,7 @@
             </geometry>
         </collision>
+        <xacro:inertial_box mass="0.5" x="0.3" y="0.3" z="0.15">
+            <origin xyz="0.15 0 0.075" rpy="0 0 0"/>
+        </xacro:inertial_box>
     </link>
     <!-- LEFT WHEEL -->
@@ -50,4 +53,7 @@
             <material name="blue"/>
         </visual>
+        <xacro:inertial_cylinder mass="0.1" length="0.05" radius="0.05">
+            <origin xyz="0 0 0" rpy="0 0 0"/>
+        </xacro:inertial_cylinder>
     </link>
     <!-- RIGHT WHEEL -->
@@ -65,4 +71,7 @@
             <material name="blue"/>
         </visual>
+        <xacro:inertial_cylinder mass="0.1" length="0.05" radius="0.05">
+            <origin xyz="0 0 0" rpy="0 0 0"/>
+        </xacro:inertial_cylinder>
     </link>
     <!-- CASTER WHEEL -->
@@ -79,4 +88,7 @@
             <material name="black"/>
         </visual>
+        <xacro:inertial_sphere mass="0.1" radius="0.05">
+            <origin xyz="0 0 0" rpy="0 0 0"/>
+        </xacro:inertial_sphere>
     </link>
 </robot>

Commit message: feat: colors for gazebo

File: description/robot_core.xacro (robot description, xacro)
@@ -39,4 +39,7 @@
         </xacro:inertial_box>
     </link>
+    <gazebo reference="chassis">
+        <material>Gazebo/White</material>
+    </gazebo>
     <!-- LEFT WHEEL -->
     <joint name="left_wheel_joint" type="continuous">
@@ -57,4 +60,7 @@
         </xacro:inertial_cylinder>
     </link>
+    <gazebo reference="left_wheel">
+        <material>Gazebo/Blue</material>
+    </gazebo>
     <!-- RIGHT WHEEL -->
     <joint name="right_wheel_joint" type="continuous">
@@ -75,4 +81,7 @@
         </xacro:inertial_cylinder>
     </link>
+    <gazebo reference="right_wheel">
+        <material>Gazebo/Blue</material>
+    </gazebo>
     <!-- CASTER WHEEL -->
     <joint name="caster_wheel_joint" type="fixed">
@@ -92,3 +101,8 @@
         </xacro:inertial_sphere>
     </link>
+    <gazebo reference="caster_wheel">
+        <material>Gazebo/Black</material>
+        <mu1 value="0.001"/>
+        <mu2 value="0.001"/>
+    </gazebo>
 </robot>

Commit message: feat: collision

File: description/robot_core.xacro (robot description, xacro)
@@ -56,5 +56,10 @@
             <material name="blue"/>
         </visual>
-        <xacro:inertial_cylinder mass="0.1" length="0.05" radius="0.05">
+        <collision>
+            <geometry>
+                <cylinder radius="0.05" length="0.04"/>
+            </geometry>
+        </collision>
+        <xacro:inertial_cylinder mass="0.1" length="0.04" radius="0.05">
             <origin xyz="0 0 0" rpy="0 0 0"/>
         </xacro:inertial_cylinder>
@@ -77,5 +82,10 @@
             <material name="blue"/>
         </visual>
-        <xacro:inertial_cylinder mass="0.1" length="0.05" radius="0.05">
+        <collision>
+            <geometry>
+                <cylinder radius="0.05" length="0.04"/>
+            </geometry>
+        </collision>
+        <xacro:inertial_cylinder mass="0.1" length="0.04" radius="0.05">
             <origin xyz="0 0 0" rpy="0 0 0"/>
         </xacro:inertial_cylinder>
@@ -97,4 +107,9 @@
             <material name="black"/>
         </visual>
+        <collision>
+            <geometry>
+                <sphere radius="0.05"/>
+            </geometry>
+        </collision>
         <xacro:inertial_sphere mass="0.1" radius="0.05">
             <origin xyz="0 0 0" rpy="0 0 0"/>

Commit message: car

File: description/robot_core.xacro (robot description, xacro)
@@ -1,5 +1,5 @@
 <?xml version="1.0"?>
-<robot xmlns:xacro="http://www.ros.org/wiki/xacro" >
-<xacro:include filename="inertia_macros.xacro" />
+<robot xmlns:xacro="http://www.ros.org/wiki/xacro">
+<xacro:include filename="inertia_macros.xacro"/>
     <material name="white">
         <color rgba="1 1 1 1"/>
@@ -25,5 +25,5 @@
             <origin xyz="0.15 0 0.075" rpy="0 0 0"/>
             <geometry>
-                <box size="0.3 0.3 0.15"/>
+                <box size="1.2 0.6 0.26"/>
             </geometry>
             <material name="white"/>
@@ -32,5 +32,5 @@
             <origin xyz="0.15 0 0.075" rpy="0 0 0"/>
             <geometry>
-                <box size="0.3 0.3 0.15"/>
+                <box size="1.2 0.6 0.26"/>
             </geometry>
         </collision>
@@ -46,5 +46,5 @@
         <parent link="base_link"/>
         <child link="left_wheel"/>
-        <origin xyz="0 0.175 0" rpy="-${pi/2} 0 0"/>
+        <origin xyz="-0.38 0.38 0" rpy="-${pi/2} 0 0"/>
         <axis xyz="0 0 1"/>
     </joint>
@@ -52,5 +52,5 @@
         <visual>
             <geometry>
-                <cylinder length="0.04" radius="0.05" />
+                <cylinder length="0.15" radius="0.17"/>
             </geometry>
             <material name="blue"/>
@@ -58,8 +58,8 @@
         <collision>
             <geometry>
-                <cylinder radius="0.05" length="0.04"/>
+                <cylinder radius="0.17" length="0.15"/>
             </geometry>
         </collision>
-        <xacro:inertial_cylinder mass="0.1" length="0.04" radius="0.05">
+        <xacro:inertial_cylinder mass="0.1" length="0.15" radius="0.17">
             <origin xyz="0 0 0" rpy="0 0 0"/>
         </xacro:inertial_cylinder>
@@ -72,5 +72,5 @@
         <parent link="base_link"/>
         <child link="right_wheel"/>
-        <origin xyz="0 -0.175 0" rpy="${pi/2} 0 0"/>
+        <origin xyz="-0.38 -0.38 0" rpy="${pi/2} 0 0"/>
         <axis xyz="0 0 -1"/>
     </joint>
@@ -78,5 +78,5 @@
         <visual>
             <geometry>
-                <cylinder length="0.04" radius="0.05" />
+                <cylinder length="0.15" radius="0.17"/>
             </geometry>
             <material name="blue"/>
@@ -84,8 +84,8 @@
         <collision>
             <geometry>
-                <cylinder radius="0.05" length="0.04"/>
+                <cylinder radius="0.17" length="0.15"/>
             </geometry>
         </collision>
-        <xacro:inertial_cylinder mass="0.1" length="0.04" radius="0.05">
+        <xacro:inertial_cylinder mass="0.1" length="0.15" radius="0.17">
             <origin xyz="0 0 0" rpy="0 0 0"/>
         </xacro:inertial_cylinder>
@@ -94,30 +94,75 @@
         <material>Gazebo/Blue</material>
     </gazebo>
-    <!-- CASTER WHEEL -->
-    <joint name="caster_wheel_joint" type="fixed">
-        <parent link="chassis"/>
-        <child link="caster_wheel"/>
-        <origin xyz="0.24 0 0" rpy="0 0 0"/>
+    <!-- BACK LEFT WHEEL -->
+    <joint name="back_left_wheel_joint" type="continuous">
+        <parent link="base_link"/>
+        <child link="back_left_wheel"/>
+        <origin xyz="0.38 0.38 0" rpy="-${pi/2} 0 0"/>
+        <axis xyz="0 0 1"/>
     </joint>
-    <link name="caster_wheel">
+    <link name="back_left_wheel">
         <visual>
             <geometry>
-                <sphere radius="0.05" />
+                <cylinder length="0.15" radius="0.17"/>
             </geometry>
-            <material name="black"/>
+            <material name="blue"/>
         </visual>
         <collision>
             <geometry>
-                <sphere radius="0.05"/>
+                <cylinder radius="0.17" length="0.15"/>
             </geometry>
         </collision>
-        <xacro:inertial_sphere mass="0.1" radius="0.05">
+        <xacro:inertial_cylinder mass="0.1" length="0.15" radius="0.17">
             <origin xyz="0 0 0" rpy="0 0 0"/>
-        </xacro:inertial_sphere>
+        </xacro:inertial_cylinder>
     </link>
-    <gazebo reference="caster_wheel">
-        <material>Gazebo/Black</material>
-        <mu1 value="0.001"/>
-        <mu2 value="0.001"/>
+    <gazebo reference="back_left_wheel">
+        <material>Gazebo/Blue</material>
+    </gazebo>
+    <!-- BACK RIGHT WHEEL -->
+    <joint name="back_right_wheel_joint" type="continuous">
+        <parent link="base_link"/>
+        <child link="back_right_wheel"/>
+        <origin xyz="0.38 -0.38 0" rpy="${pi/2} 0 0"/>
+        <axis xyz="0 0 -1"/>
+    </joint>
+    <link name="back_right_wheel">
+        <visual>
+            <geometry>
+                <cylinder length="0.15" radius="0.17"/>
+            </geometry>
+            <material name="blue"/>
+        </visual>
+        <collision>
+            <geometry>
+                <cylinder radius="0.17" length="0.15"/>
+            </geometry>
+        </collision>
+        <xacro:inertial_cylinder mass="0.1" length="0.15" radius="0.17">
+            <origin xyz="0 0 0" rpy="0 0 0"/>
+        </xacro:inertial_cylinder>
+    </link>
+    <gazebo reference="back_right_wheel">
+        <material>Gazebo/Blue</material>
+    </gazebo>
+    <!-- УПРАВЛЕНИЕ 4-КОЛЕСНЫМ РОВЕРОМ -->
+<gazebo>
+        <plugin name="skid_steer_drive" filename="libgazebo_ros_skid_steer_drive.so">
+            <commandTopic>cmd_vel</commandTopic>
+            <odometryTopic>odom</odometryTopic>
+            <odometryFrame>odom</odometryFrame>
+            <robotBaseFrame>base_link</robotBaseFrame>
+            <!-- Левый борт: переднее и заднее колесо -->
+            <leftJoint>left_wheel_joint back_left_wheel_joint</leftJoint>
+            <!-- Правый борт: переднее и заднее колесо -->
+            <rightJoint>right_wheel_joint back_right_wheel_joint</rightJoint>
+            <wheelSeparation>0.35</wheelSeparation>
+            <wheelDiameter>0.10</wheelDiameter>
+            <torque>20</torque>
+            <updateRate>50.0</updateRate>
+            <publishWheelTF>true</publishWheelTF>
+            <publishWheelJointState>true</publishWheelJointState>
+            <publishTf>true</publishTf>
+        </plugin>
     </gazebo>
 </robot>

Commit message: car

File: description/robot_core.xacro (robot description, xacro)
@@ -106,5 +106,5 @@
         <parent link="base_link"/>
         <child link="back_left_wheel"/>
-        <origin xyz="0.38 0.38 0" rpy="-${pi/2} 0 0"/>
+        <origin xyz="0.48 0.38 0" rpy="-${pi/2} 0 0"/>
         <axis xyz="0 0 1"/>
     </joint>
@@ -136,5 +136,5 @@
         <parent link="base_link"/>
         <child link="back_right_wheel"/>
-        <origin xyz="0.38 -0.38 0" rpy="${pi/2} 0 0"/>
+        <origin xyz="0.48 -0.38 0" rpy="${pi/2} 0 0"/>
         <axis xyz="0 0 -1"/>
     </joint>
