Commit message: apocalipsis

File: description/robot.urdf.xacro (robot description, xacro)
@@ -3,3 +3,51 @@
     <xacro:include filename="robot_core.xacro" />
     <xacro:include filename="gazebo_control.xacro" />
+<!-- Camera -->
+<link name="camera_link">
+  <visual>
+    <geometry>
+      <box size="0.05 0.05 0.05"/>
+    </geometry>
+  </visual>
+  <collision>
+    <geometry>
+      <box size="0.05 0.05 0.05"/>
+    </geometry>
+  </collision>
+  <inertial>
+    <mass value="0.1"/>
+    <inertia ixx="0.001" ixy="0.0" ixz="0.0" iyy="0.001" iyz="0.0" izz="0.001"/>
+  </inertial>
+</link>
+<joint name="camera_joint" type="fixed">
+  <parent link="base_link"/>
+  <child link="camera_link"/>
+  <origin xyz="0.2 0 0.1" rpy="0 0 0"/>
+</joint>
+<!-- Gazebo camera plugin -->
+<gazebo reference="camera_link">
+  <sensor type="camera" name="camera">
+    <update_rate>30.0</update_rate>
+    <camera name="main">
+      <horizontal_fov>1.047</horizontal_fov>
+      <image>
+        <width>640</width>
+        <height>480</height>
+        <format>R8G8B8</format>
+      </image>
+      <clip>
+        <near>0.05</near>
+        <far>100.0</far>
+      </clip>
+    </camera>
+    <plugin filename="libgazebo_ros_camera.so" name="camera_controller">
+      <ros>
+        <namespace>camera</namespace>
+      </ros>
+      <camera_name>camera</camera_name>
+      <frame_name>camera_link</frame_name>
+      <hack_baseline>0.07</hack_baseline>
+    </plugin>
+  </sensor>
+</gazebo>
 </robot>

Commit message: fix: fix Petya's commits

File: description/robot.urdf.xacro (robot description, xacro)
@@ -3,51 +3,3 @@
     <xacro:include filename="robot_core.xacro" />
     <xacro:include filename="gazebo_control.xacro" />
-<!-- Camera -->
-<link name="camera_link">
-  <visual>
-    <geometry>
-      <box size="0.05 0.05 0.05"/>
-    </geometry>
-  </visual>
-  <collision>
-    <geometry>
-      <box size="0.05 0.05 0.05"/>
-    </geometry>
-  </collision>
-  <inertial>
-    <mass value="0.1"/>
-    <inertia ixx="0.001" ixy="0.0" ixz="0.0" iyy="0.001" iyz="0.0" izz="0.001"/>
-  </inertial>
-</link>
-<joint name="camera_joint" type="fixed">
-  <parent link="base_link"/>
-  <child link="camera_link"/>
-  <origin xyz="0.2 0 0.1" rpy="0 0 0"/>
-</joint>
-<!-- Gazebo camera plugin -->
-<gazebo reference="camera_link">
-  <sensor type="camera" name="camera">
-    <update_rate>30.0</update_rate>
-    <camera name="main">
-      <horizontal_fov>1.047</horizontal_fov>
-      <image>
-        <width>640</width>
-        <height>480</height>
-        <format>R8G8B8</format>
-      </image>
-      <clip>
-        <near>0.05</near>
-        <far>100.0</far>
-      </clip>
-    </camera>
-    <plugin filename="libgazebo_ros_camera.so" name="camera_controller">
-      <ros>
-        <namespace>camera</namespace>
-      </ros>
-      <camera_name>camera</camera_name>
-      <frame_name>camera_link</frame_name>
-      <hack_baseline>0.07</hack_baseline>
-    </plugin>
-  </sensor>
-</gazebo>
 </robot>
